Commit message: Better trees and collisions unacceptable

File: ur_e_description/urdf/trees/envy/test/tree_14.urdf (robot description, URDF)
Before this commit: robot ur5e, 2 links, 1 joints
Links:
- link tree: geometry collision mesh filename=./ur_e_description/meshes/trees/envy/test/tree_14.obj scale=1 1 1; visual mesh filename=./ur_e_description/meshes/trees/envy/test/tree_14.obj scale=1 1 1
