Commit message: Added URDF for trees:

File: meshes_and_urdf/urdf/trees/envy/test/tree_24.urdf (robot description, URDF)
Before this commit: robot ur5e, 2 links, 1 joints
Links:
- link tree: geometry collision mesh filename=./meshes_and_urdf/meshes/trees/envy/test\tree_24.obj scale=1 1 1; visual mesh filename=./meshes_and_urdf/meshes/trees/envy/test\tree_24.obj scale=1 1 1

File: meshes_and_urdf/urdf/trees/envy/train/tree_0.urdf (robot description, URDF)
Before this commit: robot ur5e, 2 links, 1 joints
Links:
- link tree: geometry collision mesh filename=./meshes_and_urdf/meshes/trees/envy/train\tree_0.obj scale=1 1 1; visual mesh filename=./meshes_and_urdf/meshes/trees/envy/train\tree_0.obj scale=1 1 1

File: meshes_and_urdf/urdf/trees/envy/train/tree_1.urdf (robot description, URDF)
Before this commit: robot ur5e, 2 links, 1 joints
Links:
- link tree: geometry collision mesh filename=./meshes_and_urdf/meshes/trees/envy/train\tree_1.obj scale=1 1 1; visual mesh filename=./meshes_and_urdf/meshes/trees/envy/train\tree_1.obj scale=1 1 1

File: meshes_and_urdf/urdf/trees/envy/train/tree_10.urdf (robot description, URDF)
Before this commit: robot ur5e, 2 links, 1 joints
Links:
- link tree: geometry collision mesh filename=./meshes_and_urdf/meshes/trees/envy/train\tree_10.obj scale=1 1 1; visual mesh filename=./meshes_and_urdf/meshes/trees/envy/train\tree_10.obj scale=1 1 1

File: meshes_and_urdf/urdf/trees/envy/train/tree_11.urdf (robot description, URDF)
Before this commit: robot ur5e, 2 links, 1 joints
Links:
- link tree: geometry collision mesh filename=./meshes_and_urdf/meshes/trees/envy/train\tree_11.obj scale=1 1 1; visual mesh filename=./meshes_and_urdf/meshes/trees/envy/train\tree_11.obj scale=1 1 1

File: meshes_and_urdf/urdf/trees/envy/train/tree_12.urdf (robot description, URDF)
Before this commit: robot ur5e, 2 links, 1 joints
Links:
- link tree: geometry collision mesh filename=./meshes_and_urdf/meshes/trees/envy/train\tree_12.obj scale=1 1 1; visual mesh filename=./meshes_and_urdf/meshes/trees/envy/train\tree_12.obj scale=1 1 1

File: meshes_and_urdf/urdf/trees/envy/train/tree_13.urdf (robot description, URDF)
Before this commit: robot ur5e, 2 links, 1 joints
Links:
- link tree: geometry collision mesh filename=./meshes_and_urdf/meshes/trees/envy/train\tree_13.obj scale=1 1 1; visual mesh filename=./meshes_and_urdf/meshes/trees/envy/train\tree_13.obj scale=1 1 1

File: meshes_and_urdf/urdf/trees/envy/train/tree_14.urdf (robot description, URDF)
Before this commit: robot ur5e, 2 links, 1 joints
Links:
- link tree: geometry collision mesh filename=./meshes_and_urdf/meshes/trees/envy/train\tree_14.obj scale=1 1 1; visual mesh filename=./meshes_and_urdf/meshes/trees/envy/train\tree_14.obj scale=1 1 1

File: meshes_and_urdf/urdf/trees/envy/train/tree_15.urdf (robot description, URDF)
Before this commit: robot ur5e, 2 links, 1 joints
Links:
- link tree: geometry collision mesh filename=./meshes_and_urdf/meshes/trees/envy/train\tree_15.obj scale=1 1 1; visual mesh filename=./meshes_and_urdf/meshes/trees/envy/train\tree_15.obj scale=1 1 1

File: meshes_and_urdf/urdf/trees/envy/train/tree_16.urdf (robot description, URDF)
Before this commit: robot ur5e, 2 links, 1 joints
Links:
- link tree: geometry collision mesh filename=./meshes_and_urdf/meshes/trees/envy/train\tree_16.obj scale=1 1 1; visual mesh filename=./meshes_and_urdf/meshes/trees/envy/train\tree_16.obj scale=1 1 1

File: meshes_and_urdf/urdf/trees/envy/train/tree_17.urdf (robot description, URDF)
Before this commit: robot ur5e, 2 links, 1 joints
Links:
- link tree: geometry collision mesh filename=./meshes_and_urdf/meshes/trees/envy/train\tree_17.obj scale=1 1 1; visual mesh filename=./meshes_and_urdf/meshes/trees/envy/train\tree_17.obj scale=1 1 1

File: meshes_and_urdf/urdf/trees/envy/train/tree_18.urdf (robot description, URDF)
Before this commit: robot ur5e, 2 links, 1 joints
Links:
- link tree: geometry collision mesh filename=./meshes_and_urdf/meshes/trees/envy/train\tree_18.obj scale=1 1 1; visual mesh filename=./meshes_and_urdf/meshes/trees/envy/train\tree_18.obj scale=1 1 1

File: meshes_and_urdf/urdf/trees/envy/train/tree_19.urdf (robot description, URDF)
Before this commit: robot ur5e, 2 links, 1 joints
Links:
- link tree: geometry collision mesh filename=./meshes_and_urdf/meshes/trees/envy/train\tree_19.obj scale=1 1 1; visual mesh filename=./meshes_and_urdf/meshes/trees/envy/train\tree_19.obj scale=1 1 1

File: meshes_and_urdf/urdf/trees/envy/train/tree_2.urdf (robot description, URDF)
Before this commit: robot ur5e, 2 links, 1 joints
Links:
- link tree: geometry collision mesh filename=./meshes_and_urdf/meshes/trees/envy/train\tree_2.obj scale=1 1 1; visual mesh filename=./meshes_and_urdf/meshes/trees/envy/train\tree_2.obj scale=1 1 1

File: meshes_and_urdf/urdf/trees/envy/train/tree_20.urdf (robot description, URDF)
Before this commit: robot ur5e, 2 links, 1 joints
Links:
- link tree: geometry collision mesh filename=./meshes_and_urdf/meshes/trees/envy/train\tree_20.obj scale=1 1 1; visual mesh filename=./meshes_and_urdf/meshes/trees/envy/train\tree_20.obj scale=1 1 1

File: meshes_and_urdf/urdf/trees/envy/train/tree_21.urdf (robot description, URDF)
Before this commit: robot ur5e, 2 links, 1 joints
Links:
- link tree: geometry collision mesh filename=./meshes_and_urdf/meshes/trees/envy/train\tree_21.obj scale=1 1 1; visual mesh filename=./meshes_and_urdf/meshes/trees/envy/train\tree_21.obj scale=1 1 1

File: meshes_and_urdf/urdf/trees/envy/train/tree_22.urdf (robot description, URDF)
Before this commit: robot ur5e, 2 links, 1 joints
Links:
- link tree: geometry collision mesh filename=./meshes_and_urdf/meshes/trees/envy/train\tree_22.obj scale=1 1 1; visual mesh filename=./meshes_and_urdf/meshes/trees/envy/train\tree_22.obj scale=1 1 1

File: meshes_and_urdf/urdf/trees/envy/train/tree_23.urdf (robot description, URDF)
Before this commit: robot ur5e, 2 links, 1 joints
Links:
- link tree: geometry collision mesh filename=./meshes_and_urdf/meshes/trees/envy/train\tree_23.obj scale=1 1 1; visual mesh filename=./meshes_and_urdf/meshes/trees/envy/train\tree_23.obj scale=1 1 1

File: meshes_and_urdf/urdf/trees/envy/train/tree_3.urdf (robot description, URDF)
Before this commit: robot ur5e, 2 links, 1 joints
Links:
- link tree: geometry collision mesh filename=./meshes_and_urdf/meshes/trees/envy/train\tree_3.obj scale=1 1 1; visual mesh filename=./meshes_and_urdf/meshes/trees/envy/train\tree_3.obj scale=1 1 1

File: meshes_and_urdf/urdf/trees/envy/train/tree_4.urdf (robot description, URDF)
Before this commit: robot ur5e, 2 links, 1 joints
Links:
- link tree: geometry collision mesh filename=./meshes_and_urdf/meshes/trees/envy/train\tree_4.obj scale=1 1 1; visual mesh filename=./meshes_and_urdf/meshes/trees/envy/train\tree_4.obj scale=1 1 1
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
Commit message: making urdf linux friendly

File: meshes_and_urdf/urdf/trees/envy/test/tree_24.urdf (robot description, URDF)
Before this commit: robot ur5e, 2 links, 1 joints
Links:
- link tree: geometry collision mesh filename=./meshes_and_urdf/meshes/trees/envy/test/tree_24.obj scale=1 1 1; visual mesh filename=./meshes_and_urdf/meshes/trees/envy/test/tree_24.obj scale=1 1 1

File: meshes_and_urdf/urdf/trees/envy/train/tree_0.urdf (robot description, URDF)
Before this commit: robot ur5e, 2 links, 1 joints
Links:
- link tree: geometry collision mesh filename=./meshes_and_urdf/meshes/trees/envy/train/tree_0.obj scale=1 1 1; visual mesh filename=./meshes_and_urdf/meshes/trees/envy/train/tree_0.obj scale=1 1 1
