Commit message: Logging offline stuff and getting file format right

File: meshes_and_urdf/urdf/trees/envy/test/tree_0.urdf (robot description, URDF)
Before this commit: robot ur5e, 2 links, 1 joints
Links:
- link tree: geometry collision mesh filename=meshes_and_urdf/meshes/trees/envy/test/tree_0.obj scale=1 1 1; visual mesh filename=meshes_and_urdf/meshes/trees/envy/test/tree_0.obj scale=1 1 1

File: meshes_and_urdf/urdf/trees/envy/test/tree_141.urdf (robot description, URDF)
Before this commit: robot ur5e, 2 links, 1 joints
Links:
- link tree: geometry collision mesh filename=meshes_and_urdf/meshes/trees/envy/test/tree_141.obj scale=1 1 1; visual mesh filename=meshes_and_urdf/meshes/trees/envy/test/tree_141.obj scale=1 1 1

File: meshes_and_urdf/urdf/trees/envy/test/tree_142.urdf (robot description, URDF)
Before this commit: robot ur5e, 2 links, 1 joints
Links:
- link tree: geometry collision mesh filename=meshes_and_urdf/meshes/trees/envy/test/tree_142.obj scale=1 1 1; visual mesh filename=meshes_and_urdf/meshes/trees/envy/test/tree_142.obj scale=1 1 1

File: meshes_and_urdf/urdf/trees/envy/test/tree_143.urdf (robot description, URDF)
Before this commit: robot ur5e, 2 links, 1 joints
Links:
- link tree: geometry collision mesh filename=meshes_and_urdf/meshes/trees/envy/test/tree_143.obj scale=1 1 1; visual mesh filename=meshes_and_urdf/meshes/trees/envy/test/tree_143.obj scale=1 1 1

File: meshes_and_urdf/urdf/trees/envy/test/tree_144.urdf (robot description, URDF)
Before this commit: robot ur5e, 2 links, 1 joints
Links:
- link tree: geometry collision mesh filename=meshes_and_urdf/meshes/trees/envy/test/tree_144.obj scale=1 1 1; visual mesh filename=meshes_and_urdf/meshes/trees/envy/test/tree_144.obj scale=1 1 1

File: meshes_and_urdf/urdf/trees/envy/test/tree_145.urdf (robot description, URDF)
Before this commit: robot ur5e, 2 links, 1 joints
Links:
- link tree: geometry collision mesh filename=meshes_and_urdf/meshes/trees/envy/test/tree_145.obj scale=1 1 1; visual mesh filename=meshes_and_urdf/meshes/trees/envy/test/tree_145.obj scale=1 1 1

File: meshes_and_urdf/urdf/trees/envy/test/tree_146.urdf (robot description, URDF)
Before this commit: robot ur5e, 2 links, 1 joints
Links:
- link tree: geometry collision mesh filename=meshes_and_urdf/meshes/trees/envy/test/tree_146.obj scale=1 1 1; visual mesh filename=meshes_and_urdf/meshes/trees/envy/test/tree_146.obj scale=1 1 1

File: meshes_and_urdf/urdf/trees/envy/test/tree_147.urdf (robot description, URDF)
Before this commit: robot ur5e, 2 links, 1 joints
Links:
- link tree: geometry collision mesh filename=meshes_and_urdf/meshes/trees/envy/test/tree_147.obj scale=1 1 1; visual mesh filename=meshes_and_urdf/meshes/trees/envy/test/tree_147.obj scale=1 1 1

File: meshes_and_urdf/urdf/trees/envy/test/tree_148.urdf (robot description, URDF)
Before this commit: robot ur5e, 2 links, 1 joints
Links:
- link tree: geometry collision mesh filename=meshes_and_urdf/meshes/trees/envy/test/tree_148.obj scale=1 1 1; visual mesh filename=meshes_and_urdf/meshes/trees/envy/test/tree_148.obj scale=1 1 1

File: meshes_and_urdf/urdf/trees/envy/test/tree_149.urdf (robot description, URDF)
Before this commit: robot ur5e, 2 links, 1 joints
Links:
- link tree: geometry collision mesh filename=meshes_and_urdf/meshes/trees/envy/test/tree_149.obj scale=1 1 1; visual mesh filename=meshes_and_urdf/meshes/trees/envy/test/tree_149.obj scale=1 1 1

File: meshes_and_urdf/urdf/trees/envy/test/tree_150.urdf (robot description, URDF)
Before this commit: robot ur5e, 2 links, 1 joints
Links:
- link tree: geometry collision mesh filename=meshes_and_urdf/meshes/trees/envy/test/tree_150.obj scale=1 1 1; visual mesh filename=meshes_and_urdf/meshes/trees/envy/test/tree_150.obj scale=1 1 1

File: meshes_and_urdf/urdf/trees/envy/test_labelled_split/tree_0_BRANCH.urdf (robot description, URDF)
Before this commit: robot ur5e, 2 links, 1 joints
Links:
- link tree: geometry collision mesh filename=meshes_and_urdf/meshes/trees/envy/test_labelled_split/tree_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 scale=1 1 1; visual mesh filename=meshes_and_urdf/meshes/trees/envy/test_labelled_split/tree_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 scale=1 1 1

File: meshes_and_urdf/urdf/trees/envy/test_labelled_split/tree_0_SPUR.urdf (robot description, URDF)
Before this commit: robot ur5e, 2 links, 1 joints
Links:
- link tree: geometry collision mesh filename=meshes_and_urdf/meshes/trees/envy/test_labelled_split/tree_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 scale=1 1 1; visual mesh filename=meshes_and_urdf/meshes/trees/envy/test_labelled_split/tree_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 scale=1 1 1

File: meshes_and_urdf/urdf/trees/envy/test_labelled_split/tree_0_TRUNK.urdf (robot description, URDF)
Before this commit: robot ur5e, 2 links, 1 joints
Links:
- link tree: geometry collision mesh filename=meshes_and_urdf/meshes/trees/envy/test_labelled_split/tree_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 scale=1 1 1; visual mesh filename=meshes_and_urdf/meshes/trees/envy/test_labelled_split/tree_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 scale=1 1 1

File: meshes_and_urdf/urdf/trees/envy/test_labelled_split/tree_0_WATER_BRANCH.urdf (robot description, URDF)
Before this commit: robot ur5e, 2 links, 1 joints
Links:
- link tree: geometry collision mesh filename=meshes_and_urdf/meshes/trees/envy/test_labelled_split/tree_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 scale=1 1 1; visual mesh filename=meshes_and_urdf/meshes/trees/envy/test_labelled_split/tree_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 scale=1 1 1

File: meshes_and_urdf/urdf/trees/envy/test_labelled_split/tree_141_BRANCH.urdf (robot description, URDF)
Before this commit: robot ur5e, 2 links, 1 joints
Links:
- link tree: geometry collision mesh filename=meshes_and_urdf/meshes/trees/envy/test_labelled_split/tree_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 scale=1 1 1; visual mesh filename=meshes_and_urdf/meshes/trees/envy/test_labelled_split/tree_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 scale=1 1 1

File: meshes_and_urdf/urdf/trees/envy/test_labelled_split/tree_141_SPUR.urdf (robot description, URDF)
Before this commit: robot ur5e, 2 links, 1 joints
Links:
- link tree: geometry collision mesh filename=meshes_and_urdf/meshes/trees/envy/test_labelled_split/tree_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 scale=1 1 1; visual mesh filename=meshes_and_urdf/meshes/trees/envy/test_labelled_split/tree_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 scale=1 1 1

File: meshes_and_urdf/urdf/trees/envy/test_labelled_split/tree_141_TRUNK.urdf (robot description, URDF)
Before this commit: robot ur5e, 2 links, 1 joints
Links:
- link tree: geometry collision mesh filename=meshes_and_urdf/meshes/trees/envy/test_labelled_split/tree_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 scale=1 1 1; visual mesh filename=meshes_and_urdf/meshes/trees/envy/test_labelled_split/tree_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 scale=1 1 1

File: meshes_and_urdf/urdf/trees/envy/test_labelled_split/tree_141_WATER_BRANCH.urdf (robot description, URDF)
Before this commit: robot ur5e, 2 links, 1 joints
Links:
- link tree: geometry collision mesh filename=meshes_and_urdf/meshes/trees/envy/test_labelled_split/tree_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 scale=1 1 1; visual mesh filename=meshes_and_urdf/meshes/trees/envy/test_labelled_split/tree_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 scale=1 1 1

File: meshes_and_urdf/urdf/trees/envy/test_labelled_split/tree_142_BRANCH.urdf (robot description, URDF)
Before this commit: robot ur5e, 2 links, 1 joints
Links:
- link tree: geometry collision mesh filename=meshes_and_urdf/meshes/trees/envy/test_labelled_split/tree_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 scale=1 1 1; visual mesh filename=meshes_and_urdf/meshes/trees/envy/test_labelled_split/tree_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 scale=1 1 1
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