Commit message: remove divide by 0 error

File: meshes_and_urdf/urdf/trees/envy/train/tree_1.urdf (robot description, URDF)
Before this commit: robot ur5e, 2 links, 1 joints
Links:
- link tree: geometry collision mesh filename=meshes_and_urdf\meshes\trees\envy\train\tree_1.obj scale=1 1 1; visual mesh filename=meshes_and_urdf\meshes\trees\envy\train\tree_1.obj scale=1 1 1

File: meshes_and_urdf/urdf/trees/envy/train/tree_10.urdf (robot description, URDF)
Before this commit: robot ur5e, 2 links, 1 joints
Links:
- link tree: geometry collision mesh filename=meshes_and_urdf\meshes\trees\envy\train\tree_10.obj scale=1 1 1; visual mesh filename=meshes_and_urdf\meshes\trees\envy\train\tree_10.obj scale=1 1 1

File: meshes_and_urdf/urdf/trees/envy/train/tree_100.urdf (robot description, URDF)
Before this commit: robot ur5e, 2 links, 1 joints
Links:
- link tree: geometry collision mesh filename=meshes_and_urdf\meshes\trees\envy\train\tree_100.obj scale=1 1 1; visual mesh filename=meshes_and_urdf\meshes\trees\envy\train\tree_100.obj scale=1 1 1

File: meshes_and_urdf/urdf/trees/envy/train/tree_101.urdf (robot description, URDF)
Before this commit: robot ur5e, 2 links, 1 joints
Links:
- link tree: geometry collision mesh filename=meshes_and_urdf\meshes\trees\envy\train\tree_101.obj scale=1 1 1; visual mesh filename=meshes_and_urdf\meshes\trees\envy\train\tree_101.obj scale=1 1 1

File: meshes_and_urdf/urdf/trees/envy/train/tree_102.urdf (robot description, URDF)
Before this commit: robot ur5e, 2 links, 1 joints
Links:
- link tree: geometry collision mesh filename=meshes_and_urdf\meshes\trees\envy\train\tree_102.obj scale=1 1 1; visual mesh filename=meshes_and_urdf\meshes\trees\envy\train\tree_102.obj scale=1 1 1

File: meshes_and_urdf/urdf/trees/envy/train/tree_103.urdf (robot description, URDF)
Before this commit: robot ur5e, 2 links, 1 joints
Links:
- link tree: geometry collision mesh filename=meshes_and_urdf\meshes\trees\envy\train\tree_103.obj scale=1 1 1; visual mesh filename=meshes_and_urdf\meshes\trees\envy\train\tree_103.obj scale=1 1 1

File: meshes_and_urdf/urdf/trees/envy/train/tree_104.urdf (robot description, URDF)
Before this commit: robot ur5e, 2 links, 1 joints
Links:
- link tree: geometry collision mesh filename=meshes_and_urdf\meshes\trees\envy\train\tree_104.obj scale=1 1 1; visual mesh filename=meshes_and_urdf\meshes\trees\envy\train\tree_104.obj scale=1 1 1

File: meshes_and_urdf/urdf/trees/envy/train/tree_105.urdf (robot description, URDF)
Before this commit: robot ur5e, 2 links, 1 joints
Links:
- link tree: geometry collision mesh filename=meshes_and_urdf\meshes\trees\envy\train\tree_105.obj scale=1 1 1; visual mesh filename=meshes_and_urdf\meshes\trees\envy\train\tree_105.obj scale=1 1 1

File: meshes_and_urdf/urdf/trees/envy/train/tree_106.urdf (robot description, URDF)
Before this commit: robot ur5e, 2 links, 1 joints
Links:
- link tree: geometry collision mesh filename=meshes_and_urdf\meshes\trees\envy\train\tree_106.obj scale=1 1 1; visual mesh filename=meshes_and_urdf\meshes\trees\envy\train\tree_106.obj scale=1 1 1

File: meshes_and_urdf/urdf/trees/envy/train/tree_107.urdf (robot description, URDF)
Before this commit: robot ur5e, 2 links, 1 joints
Links:
- link tree: geometry collision mesh filename=meshes_and_urdf\meshes\trees\envy\train\tree_107.obj scale=1 1 1; visual mesh filename=meshes_and_urdf\meshes\trees\envy\train\tree_107.obj scale=1 1 1

File: meshes_and_urdf/urdf/trees/envy/train/tree_108.urdf (robot description, URDF)
Before this commit: robot ur5e, 2 links, 1 joints
Links:
- link tree: geometry collision mesh filename=meshes_and_urdf\meshes\trees\envy\train\tree_108.obj scale=1 1 1; visual mesh filename=meshes_and_urdf\meshes\trees\envy\train\tree_108.obj scale=1 1 1

File: meshes_and_urdf/urdf/trees/envy/train/tree_109.urdf (robot description, URDF)
Before this commit: robot ur5e, 2 links, 1 joints
Links:
- link tree: geometry collision mesh filename=meshes_and_urdf\meshes\trees\envy\train\tree_109.obj scale=1 1 1; visual mesh filename=meshes_and_urdf\meshes\trees\envy\train\tree_109.obj scale=1 1 1

File: meshes_and_urdf/urdf/trees/envy/train/tree_11.urdf (robot description, URDF)
Before this commit: robot ur5e, 2 links, 1 joints
Links:
- link tree: geometry collision mesh filename=meshes_and_urdf\meshes\trees\envy\train\tree_11.obj scale=1 1 1; visual mesh filename=meshes_and_urdf\meshes\trees\envy\train\tree_11.obj scale=1 1 1

File: meshes_and_urdf/urdf/trees/envy/train/tree_110.urdf (robot description, URDF)
Before this commit: robot ur5e, 2 links, 1 joints
Links:
- link tree: geometry collision mesh filename=meshes_and_urdf\meshes\trees\envy\train\tree_110.obj scale=1 1 1; visual mesh filename=meshes_and_urdf\meshes\trees\envy\train\tree_110.obj scale=1 1 1

File: meshes_and_urdf/urdf/trees/envy/train/tree_111.urdf (robot description, URDF)
Before this commit: robot ur5e, 2 links, 1 joints
Links:
- link tree: geometry collision mesh filename=meshes_and_urdf\meshes\trees\envy\train\tree_111.obj scale=1 1 1; visual mesh filename=meshes_and_urdf\meshes\trees\envy\train\tree_111.obj scale=1 1 1

File: meshes_and_urdf/urdf/trees/envy/train/tree_112.urdf (robot description, URDF)
Before this commit: robot ur5e, 2 links, 1 joints
Links:
- link tree: geometry collision mesh filename=meshes_and_urdf\meshes\trees\envy\train\tree_112.obj scale=1 1 1; visual mesh filename=meshes_and_urdf\meshes\trees\envy\train\tree_112.obj scale=1 1 1

File: meshes_and_urdf/urdf/trees/envy/train/tree_113.urdf (robot description, URDF)
Before this commit: robot ur5e, 2 links, 1 joints
Links:
- link tree: geometry collision mesh filename=meshes_and_urdf\meshes\trees\envy\train\tree_113.obj scale=1 1 1; visual mesh filename=meshes_and_urdf\meshes\trees\envy\train\tree_113.obj scale=1 1 1

File: meshes_and_urdf/urdf/trees/envy/train/tree_114.urdf (robot description, URDF)
Before this commit: robot ur5e, 2 links, 1 joints
Links:
- link tree: geometry collision mesh filename=meshes_and_urdf\meshes\trees\envy\train\tree_114.obj scale=1 1 1; visual mesh filename=meshes_and_urdf\meshes\trees\envy\train\tree_114.obj scale=1 1 1

File: meshes_and_urdf/urdf/trees/envy/train/tree_115.urdf (robot description, URDF)
Before this commit: robot ur5e, 2 links, 1 joints
Links:
- link tree: geometry collision mesh filename=meshes_and_urdf\meshes\trees\envy\train\tree_115.obj scale=1 1 1; visual mesh filename=meshes_and_urdf\meshes\trees\envy\train\tree_115.obj scale=1 1 1

File: meshes_and_urdf/urdf/trees/envy/train/tree_116.urdf (robot description, URDF)
Before this commit: robot ur5e, 2 links, 1 joints
Links:
- link tree: geometry collision mesh filename=meshes_and_urdf\meshes\trees\envy\train\tree_116.obj scale=1 1 1; visual mesh filename=meshes_and_urdf\meshes\trees\envy\train\tree_116.obj scale=1 1 1
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