Commit message: adding xy start

File: meshes_and_urdf/urdf/ur5e/ur5e_cutter_new_calibrated_precise_level.urdf (robot description, URDF)
Before this commit: robot ur5e, 16 links, 15 joints
Links:
- link mount: geometry visual mesh filename=ur5e/visual/robot_cart.obj

Commit message: Fixing end point of cutter

File: meshes_and_urdf/urdf/ur5e/ur5e_cutter_new_calibrated_precise_level.urdf (robot description, URDF)
Before this commit: robot ur5e, 16 links, 15 joints
Joints:
- joint cutpoint: origin xyz=0 0 0 rpy=0 0 0 -> xyz=0 0.01 0.05 rpy=0 0 0

Commit message: Adding success zone to urdf and updating termination

File: meshes_and_urdf/urdf/ur5e/ur5e_cutter_new_calibrated_precise_level.urdf (robot description, URDF)
Before this commit: robot ur5e, 16 links, 15 joints
Links:
- added link cutter_mouth; collision mesh filename=ur5e/collision/cutter-mouth-collision.stl
Joints:
- added joint cutter_mouth: type fixed, parent endpoint, child cutter_mouth, origin xyz=0 0 0 rpy=0 0 0
- joint cutpoint: origin xyz=0 0.01 0.05 rpy=0 0 0 -> xyz=0 0.01 0.04 rpy=0 0 0

Commit message: Scale reward by init, correct camera

File: meshes_and_urdf/urdf/ur5e/ur5e_cutter_new_calibrated_precise_level.urdf (robot description, URDF)
Before this commit: robot ur5e, 17 links, 16 joints
Links:
- link cutter_mouth: geometry collision mesh filename=ur5e/collision/cutter-mouth-collision.stl; visual mesh filename=ur5e/collision/cutter-mouth-collision.stl

Commit message: Added new trees

File: meshes_and_urdf/urdf/ur5e/ur5e_cutter_new_calibrated_precise_level.urdf (robot description, URDF)
Before this commit: robot ur5e, 17 links, 16 joints
Links:
- link cutter: geometry collision mesh filename=ur5e/collision/cutter_top_mount_for_rotation.obj scale=1.0 1.0 1.0; visual mesh filename=ur5e/visual/cutter_top_mount_for_rotation.obj scale=1.0 1.0 1.0
- link mount: geometry collision box size=0.5 0.5 0.75711; visual mesh filename=ur5e/visual/robot_cart.obj

Commit message: Needs refactor

File: meshes_and_urdf/urdf/ur5e/ur5e_cutter_new_calibrated_precise_level.urdf (robot description, URDF)
Before this commit: robot ur5e, 17 links, 16 joints
Links:
- link cutpoint: geometry visual sphere radius=0.01
- link endpoint: geometry visual sphere radius=0.01
Joints:
- joint endpoint: origin xyz=-0.063175 0 0.12864 rpy=0 0 0 -> xyz=0.063175 0 0.12864 rpy=0 0 0

Commit message: Adding inerital to cutter mouth to remove pyb warning

File: meshes_and_urdf/urdf/ur5e/ur5e_cutter_new_calibrated_precise_level.urdf (robot description, URDF)
Before this commit: robot ur5e, 17 links, 16 joints
Links:
- link cutter_mouth: mass None -> 1.0E-08
